File: TP4056_18650.sch (EAGLE design)
At the start: 17 parts, among them X1 USB MICRO

Commit message: .
Parts:
- added C3: 100n, rcl:C-EUC0805
Connections:
- removed net N$6: R5.1, VT1B.S
- net +3V7: now also C3.1
- net GND: now also C3.2, R5.1, VT1B.S
Changed lines of the file:
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@@
 <part name="B+" library="TP4056_18650" deviceset="B-" device=""/>
 <part name="FRAME1" library="frames" deviceset="A5L-LOC" device=""/>
+<part name="GND6" library="supply1" deviceset="GND" device=""/>
+<part name="C3" library="rcl" deviceset="C-EU" device="C0805" value="100n"/>
+<part name="GND7" library="supply1" deviceset="GND" device=""/>
 </parts>
 <sheets>
@@
 <instances>
 <instance part="DA1" gate="G$1" x="66.04" y="101.6"/>
-<instance part="+3V1" gate="G$1" x="101.6" y="63.5" smashed="yes">
-<attribute name="VALUE" x="104.14" y="66.04" size="1.778" layer="96" rot="R180"/>
+<instance part="+3V1" gate="G$1" x="101.6" y="83.82" smashed="yes">
+<attribute name="VALUE" x="104.14" y="86.36" size="1.778" layer="96" rot="R180"/>
 </instance>
 <instance part="R1" gate="G$1" x="50.8" y="116.84" smashed="yes" rot="R90">
@@
 <instance part="B+" gate="G$1" x="104.14" y="50.8"/>
 <instance part="FRAME1" gate="G$1" x="2.54" y="2.54"/>
+<instance part="GND6" gate="1" x="43.18" y="22.86"/>
+<instance part="C3" gate="G$1" x="101.6" y="73.66"/>
+<instance part="GND7" gate="1" x="101.6" y="63.5"/>
 </instances>
 <busses>
@@
 <wire x1="88.9" y1="38.1" x2="91.44" y2="38.1" width="0.1524" layer="91"/>
 </segment>
+<segment>
+<pinref part="VT1" gate="B" pin="S"/>
+<wire x1="43.18" y1="30.48" x2="43.18" y2="27.94" width="0.1524" layer="91"/>
+<wire x1="43.18" y1="27.94" x2="33.02" y2="27.94" width="0.1524" layer="91"/>
+<pinref part="R5" gate="G$1" pin="1"/>
+<wire x1="33.02" y1="27.94" x2="33.02" y2="35.56" width="0.1524" layer="91"/>
+<pinref part="GND6" gate="1" pin="GND"/>
+<wire x1="43.18" y1="25.4" x2="43.18" y2="27.94" width="0.1524" layer="91"/>
+<junction x="43.18" y="27.94"/>
+</segment>
+<segment>
+<pinref part="C3" gate="G$1" pin="2"/>
+<pinref part="GND7" gate="1" pin="GND"/>
+<wire x1="101.6" y1="68.58" x2="101.6" y2="66.04" width="0.1524" layer="91"/>
+</segment>
 </net>
 <net name="N$1" class="0">
@@
 </segment>
 </net>
-<net name="N$6" class="0">
-<segment>
-<pinref part="VT1" gate="B" pin="S"/>
-<wire x1="43.18" y1="30.48" x2="43.18" y2="27.94" width="0.1524" layer="91"/>
-<wire x1="43.18" y1="27.94" x2="33.02" y2="27.94" width="0.1524" layer="91"/>
-<pinref part="R5" gate="G$1" pin="1"/>
-<wire x1="33.02" y1="27.94" x2="33.02" y2="35.56" width="0.1524" layer="91"/>
-</segment>
-</net>
 <net name="N$7" class="0">
 <segment>
@@
 <pinref part="R6" gate="G$1" pin="2"/>
 <wire x1="93.98" y1="50.8" x2="96.52" y2="50.8" width="0.1524" layer="91"/>
-<wire x1="96.52" y1="50.8" x2="101.6" y2="50.8" width="0.1524" layer="91"/>
-<wire x1="101.6" y1="50.8" x2="101.6" y2="60.96" width="0.1524" layer="91"/>
+<wire x1="96.52" y1="50.8" x2="104.14" y2="50.8" width="0.1524" layer="91"/>
 <pinref part="+3V1" gate="G$1" pin="+3V3"/>
 <pinref part="DA1" gate="G$1" pin="BAT"/>
+<wire x1="101.6" y1="78.74" x2="101.6" y2="81.28" width="0.1524" layer="91"/>
 <wire x1="88.9" y1="91.44" x2="96.52" y2="91.44" width="0.1524" layer="91"/>
-<wire x1="96.52" y1="91.44" x2="96.52" y2="50.8" width="0.1524" layer="91"/>
+<wire x1="96.52" y1="91.44" x2="96.52" y2="78.74" width="0.1524" layer="91"/>
 <junction x="96.52" y="50.8"/>
-<wire x1="101.6" y1="50.8" x2="104.14" y2="50.8" width="0.1524" layer="91"/>
-<junction x="101.6" y="50.8"/>
+<wire x1="96.52" y1="78.74" x2="96.52" y2="50.8" width="0.1524" layer="91"/>
 <pinref part="B+" gate="G$1" pin="B-"/>
-</segment>
-</net>
+<wire x1="101.6" y1="78.74" x2="96.52" y2="78.74" width="0.1524" layer="91"/>
+<pinref part="C3" gate="G$1" pin="1"/>
+<wire x1="101.6" y1="78.74" x2="101.6" y2="76.2" width="0.1524" layer="91"/>
+<junction x="96.52" y="78.74"/>
+<junction x="101.6" y="78.74"/>
+</segment>
+</net>
